File: KiCad/MiniVCA 1.1/MiniVCA 1.1.kicad_pcb (KiCad board)
At the start: 2 copper layers, 64 x 128.5 mm, 42 parts, among them J1 CV_2, J2 CV_1, J3 AudioIn, J4 AudioOut, J5 JST_BUS, J6 IDC_BUS, J7 BOARD1_HEADERS, J8 BOARD2_HEADERS, Q1 BC559, U1 LM13700, U2 TL072

Commit message: Added rev1.1
Parts:
- U1: footprint Package_DIP:DIP-16_W10.16mm_LongPads -> Package_DIP:DIP-16_W7.62mm_LongPads
- moved U1 0.73 mm to (105.3, 134.8)
Routing:
- net Net-(R5-Pad2): track 14.4 -> 16.0 mm
- net Net-(R6-Pad1): track 31.3 -> 32.4 mm
- net Net-(C6-Pad2): track 61.1 -> 62.0 mm
- net B2_12V: track 132.4 -> 131.5 mm
- net Net-(Q1-Pad1): track 35.0 -> 35.7 mm
- net -12V: track 115.6 -> 116.2 mm
Other:
- board text added: "rev 1.1"
- board text removed: "rev 1.0"
